File: pcb/SG3525_Rev01.kicad_pcb (KiCad board)
At the start: 2 copper layers, 50 x 30 mm, 21 parts, among them J1 Conn_01x06, U1 SG3525

Commit message: pcb update
Parts:
- moved C1 78.3 mm to (138.8, 87.0)
- moved C2 78.3 mm to (148.7, 90.0)
- moved C3 78.3 mm to (153.0, 90.6)
- moved D1 78.3 mm to (138.9, 89.5)
- moved FID1 78.3 mm to (148.0, 84.0)
- moved FID2 78.3 mm to (130.5, 108.5)
- moved FID3 78.3 mm to (165.5, 108.5)
- moved H1 78.3 mm to (126.0, 109.0)
- moved H2 78.3 mm to (170.0, 109.0)
- moved H3 78.3 mm to (170.0, 85.0)
- moved H4 78.3 mm to (126.0, 85.0)
- moved J1 78.3 mm to (128.0, 104.5)
- moved JP1 78.3 mm to (133.0, 97.0)
- moved JP2 78.3 mm to (138.0, 104.5)
- moved JP3 78.3 mm to (138.0, 97.0)
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Routing:
- net Net-(U1-Pad1): track 19.0 -> 18.4 mm

Commit message: Añado archivos de fabricación, últimos detalles despues de la presentación
Routing:
- added copper zone on B.Cu, net GND
Other:
- board text added: "Minimos (Fabricante) : 10mils Grillas : 1mm , 0.5 Via: 0.8 mm / 0.4 mm Margen : 0.5 mm Pista : 1.2 mm / 1 mm / 0.8 mm Distancia a borde : 0.5mm Terminación : HASL"
Changed lines of the file:
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@@
   (general
     (thickness 1.6)
-    (drawings 10)
+    (drawings 11)
     (tracks 102)
     (zones 0)
@@
   )
   (setup
-    (last_trace_width 0.8)
+    (last_trace_width 0.25)
     (user_trace_width 0.8)
     (user_trace_width 1)
@@
     (via_min_size 0.4)
     (via_min_drill 0.3)
-    (user_via 1.6 0.8)
-    (user_via 2 1)
+    (user_via 0.8 0.4)
     (uvia_size 0.3)
     (uvia_drill 0.1)
@@
     (visible_elements FFFFFF7F)
     (pcbplotparams
-      (layerselection 0x010fc_ffffffff)
+      (layerselection 0x311f8_ffffffff)
       (usegerberextensions false)
       (usegerberattributes true)
       (usegerberadvancedattributes true)
       (creategerberjobfile true)
-      (excludeedgelayer true)
+      (excludeedgelayer false)
       (linewidth 0.100000)
       (plotframeref false)
@@
       (outputformat 1)
       (mirror false)
-      (drillshape 1)
+      (drillshape 0)
       (scaleselection 1)
-      (outputdirectory ""))
+      (outputdirectory "Gerber/"))
   )
   (net 0 "")
@@
       (effects (font (size 0.4 0.4) (thickness 0.06)))
     )
-    (pad 2 smd roundrect (at 0.7125 0 180) (size 1.075 1.05) (layers F.Cu F.Paste F.Mask) (roundrect_rratio 0.238095)
-      (net 2 GND))
-    (pad 1 smd roundrect (at -0.7125 0 180) (size 1.075 1.05) (layers F.Cu F.Paste F.Mask) (roundrect_rratio 0.238095)
+    (pad 2 smd roundrect (at 0.7125 0 180) (size 1.075 1.05) (layers F.Cu F.Paste F.Mask) (roundrect_rratio 0.2380942857142857)
+      (net 2 GND))
+    (pad 1 smd roundrect (at -0.7125 0 180) (size 1.075 1.05) (layers F.Cu F.Paste F.Mask) (roundrect_rratio 0.2380942857142857)
       (net 3 "Net-(C2-Pad1)"))
     (model ${KISYS3DMOD}/Capacitor_Tantalum_SMD.3dshapes/CP_EIA-1608-10_AVX-L.wrl
@@
       (effects (font (size 0.4 0.4) (thickness 0.06)))
     )
-    (pad 1 smd roundrect (at -0.7125 0 90) (size 1.075 1.05) (layers F.Cu F.Paste F.Mask) (roundrect_rratio 0.238095)
+    (pad 1 smd roundrect (at -0.7125 0 90) (size 1.075 1.05) (layers F.Cu F.Paste F.Mask) (roundrect_rratio 0.2380942857142857)
       (net 4 "Net-(C3-Pad1)"))
-    (pad 2 smd roundrect (at 0.7125 0 90) (size 1.075 1.05) (layers F.Cu F.Paste F.Mask) (roundrect_rratio 0.238095)
+    (pad 2 smd roundrect (at 0.7125 0 90) (size 1.075 1.05) (layers F.Cu F.Paste F.Mask) (roundrect_rratio 0.2380942857142857)
       (net 2 GND))
     (model ${KISYS3DMOD}/Capacitor_Tantalum_SMD.3dshapes/CP_EIA-1608-10_AVX-L.wrl
@@
       (effects (font (size 0.5 0.5) (thickness 0.08)))
     )
-    (pad 1 smd roundrect (at -0.9125 0 270) (size 1.025 1.4) (layers F.Cu F.Paste F.Mask) (roundrect_rratio 0.243902)
+    (pad 1 smd roundrect (at -0.9125 0 270) (size 1.025 1.4) (layers F.Cu F.Paste F.Mask) (roundrect_rratio 0.2439014634146341)
       (net 1 VCC))
-    (pad 2 smd roundrect (at 0.9125 0 270) (size 1.025 1.4) (layers F.Cu F.Paste F.Mask) (roundrect_rratio 0.243902)
+    (pad 2 smd roundrect (at 0.9125 0 270) (size 1.025 1.4) (layers F.Cu F.Paste F.Mask) (roundrect_rratio 0.2439014634146341)
       (net 5 "Net-(D1-Pad2)"))
     (model ${KISYS3DMOD}/Resistor_SMD.3dshapes/R_0805_2012Metric.wrl
@@
       (effects (font (size 0.5 0.5) (thickness 0.08)))
     )
-    (pad 1 smd roundrect (at -0.9125 0) (size 1.025 1.4) (layers F.Cu F.Paste F.Mask) (roundrect_rratio 0.243902)
+    (pad 1 smd roundrect (at -0.9125 0) (size 1.025 1.4) (layers F.Cu F.Paste F.Mask) (roundrect_rratio 0.2439014634146341)
       (net 11 "Net-(R2-Pad1)"))
-    (pad 2 smd roundrect (at 0.9125 0) (size 1.025 1.4) (layers F.Cu F.Paste F.Mask) (roundrect_rratio 0.243902)
+    (pad 2 smd roundrect (at 0.9125 0) (size 1.025 1.4) (layers F.Cu F.Paste F.Mask) (roundrect_rratio 0.2439014634146341)
       (net 12 "Net-(R2-Pad2)"))
     (model ${KISYS3DMOD}/Resistor_SMD.3dshapes/R_0805_2012Metric.wrl
@@
       (effects (font (size 0.5 0.5) (thickness 0.08)))
     )
-    (pad 2 smd roundrect (at 0.9125 0 180) (size 1.025 1.4) (layers F.Cu F.Paste F.Mask) (roundrect_rratio 0.243902)
+    (pad 2 smd roundrect (at 0.9125 0 180) (size 1.025 1.4) (layers F.Cu F.Paste F.Mask) (roundrect_rratio 0.2439014634146341)
       (net 9 "Net-(JP2-Pad2)"))
-    (pad 1 smd roundrect (at -0.9125 0 180) (size 1.025 1.4) (layers F.Cu F.Paste F.Mask) (roundrect_rratio 0.243902)
+    (pad 1 smd roundrect (at -0.9125 0 180) (size 1.025 1.4) (layers F.Cu F.Paste F.Mask) (roundrect_rratio 0.2439014634146341)
       (net 7 /PWM))
     (model ${KISYS3DMOD}/Resistor_SMD.3dshapes/R_0805_2012Metric.wrl
@@
     )
   )
+  (gr_text "Minimos (Fabricante) : 10mils\nGrillas : 1mm , 0.5\nVia:  0.8 mm / 0.4 mm\nMargen : 0.5 mm \nPista : 1.2 mm  / 1 mm / 0.8 mm\nDistancia a borde : 0.5mm\nTerminación :  HASL\n" (at 181.5 87.5) (layer Dwgs.User)
+    (effects (font (size 1 1) (thickness 0.15)) (justify left))
+  )
   (dimension 50 (width 0.15) (layer Dwgs.User)
     (gr_text "50,000 mm" (at 148 117.3) (layer Dwgs.User)
@@
   (segment (start 143.39 101.11) (end 144.85 101.11) (width 0.8) (layer F.Cu) (net 1))
   (segment (start 140 104.5) (end 143.39 101.11) (width 0.8) (layer F.Cu) (net 1))
+  (segment (start 154.5 109.5) (end 154 110) (width 0.8) (layer B.Cu) (net 1))
+  (segment (start 154 110) (end 142 110) (width 0.8) (layer B.Cu) (net 1))
+  (segment (start 142 110) (end 138 106) (width 0.8) (layer B.Cu) (net 1))
+  (segment (start 144.675 86.5) (end 154.5 86.5) (width 0.8) (layer F.Cu) (net 1))
+  (segment (start 143.5 87.675) (end 144.675 86.5) (width 0.8) (layer F.Cu) (net 1))
+  (segment (start 154.5 86.5) (end 154.5 109.5) (width 0.8) (layer B.Cu) (net 1))
+  (via (at 154.5 86.5) (size 0.8) (drill 0.4) (layers F.Cu B.Cu) (net 1))
+  (segment (start 138 106) (end 138 104.5) (width 0.8) (layer B.Cu) (net 1))
   (segment (start 128 104.5) (end 128 105.5) (width 0.8) (layer B.Cu) (net 1))
-  (segment (start 128 105.5) (end 129.5 107) (width 0.8) (layer B.Cu) (net 1))
-  (segment (start 129.5 107) (end 137 107) (width 0.8) (layer B.Cu) (net 1))
-  (segment (start 138 106) (end 138 104.5) (width 0.8) (layer B.Cu) (net 1))
-  (segment (start 137 107) (end 138 106) (width 0.8) (layer B.Cu) (net 1))
-  (segment (start 143.5 87.675) (end 144.675 86.5) (width 0.8) (layer F.Cu) (net 1))
-  (via (at 154.5 86.5) (size 0.8) (drill 0.4) (layers F.Cu B.Cu) (net 1))
-  (segment (start 144.675 86.5) (end 154.5 86.5) (width 0.8) (layer F.Cu) (net 1))
-  (segment (start 142 110) (end 138 106) (width 0.8) (layer B.Cu) (net 1))
-  (segment (start 154 110) (end 142 110) (width 0.8) (layer B.Cu) (net 1))
-  (segment (start 154.5 109.5) (end 154 110) (width 0.8) (layer B.Cu) (net 1))
-  (segment (start 154.5 86.5) (end 154.5 109.5) (width 0.8) (layer B.Cu) (net 1))
-  (segment (start 128 91.8) (end 128 94.34) (width 1.2) (layer B.Cu) (net 2))
+  (segment (start 128 105.5) (end 129 106.5) (width 0.8) (layer B.Cu) (net 1))
+  (segment (start 137.5 106.5) (end 138 106) (width 0.8) (layer B.Cu) (net 1))
+  (segment (start 129 106.5) (end 137.5 106.5) (width 0.8) (layer B.Cu) (net 1))
   (segment (start 128.12 94.46) (end 128 94.34) (width 1.2) (layer B.Cu) (net 2))
   (segment (start 133 94.46) (end 128.12 94.46) (width 1.2) (layer B.Cu) (net 2))
@@
   (segment (start 148 90) (end 148 94) (width 0.8) (layer F.Cu) (net 2))
   (segment (start 167 91.5) (end 167 99) (width 1) (layer B.Cu) (net 2))
+  (segment (start 128 94.34) (end 128 91.8) (width 1.2) (layer B.Cu) (net 2))
   (segment (start 151.15 97.3) (end 148.8 97.3) (width 0.8) (layer F.Cu) (net 3))
   (segment (start 148.8 95.67) (end 149.7 94.77) (width 0.8) (layer F.Cu) (net 3))
@@
   (segment (start 144.85 92.65) (end 146 91.5) (width 0.8) (layer F.Cu) (net 14))
   (segment (start 144.85 93.49) (end 144.85 92.65) (width 0.8) (layer F.Cu) (net 14))
+  (zone (net 2) (net_name GND) (layer B.Cu) (hatch edge 0.508)
+    (connect_pads (clearance 0.5))
+    (min_thickness 0.254)
+    (fill yes (arc_segments 32) (thermal_gap 0.5) (thermal_bridge_width 0.5))
+    (polygon
+      (pts
+        (xy 172.5 111.5) (xy 123.5 111.5) (xy 123.5 82.5) (xy 172.5 82.5)
+      )
+    )
+  )
 )
